File: UPS-2.sch (KiCad schematic (older format))
At the start: 62 parts, among them J1 PJ-102A, J2 Screw_Terminal, J3 OX40HAT, J4 Mode, J5 Ports, J6 Conn_01x05, Q1 DMG2305UX, Q2 DMMT5401, SW1 6x6mm, U1 TPS56339DDCR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

Commit message: readme + schematic update
Parts:
- R14: value 220k -> 510k
- R16: value 27k -> 62k
Connections:
- wire segments 231 -> 232
Other:
- note added: ""IDEAL DIODE""
- note added: "DEBUG CONNECTOR"
- note added: "HAT EEPROM"
- note added: "HEADER / CONNECTOR"
- note added: "INPUT SELECTOR"
- note added: "SYSTEM CONTROLLER"
- note added: "VOLTAGE REGULATORS"
- note added: "VOLTAGE SCALER"
- note added: "Vx = Vin * R16/(R14+R16) = Vin * 0.109\n--> Vin: 7.39mV / Bit"
- note removed: "Vx = Vin * R1r/(R14+R16) = Vin * 0.109\n--> Vin: m7.39mV / Bit"
- moved on the sheet: C12, C13, C14, C15, D5, D6, D7, J3, J4, J5, J6, R14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
